File: IIsi-to-ztex/hdmi.sch (KiCad schematic (older format))
At the start: 10 parts, among them J3 10029449-111RLF (HDMI A), U12 TPD12S016PWR

Commit message: cleanup DRC
Parts:
- added C24: 100nF, Capacitor_SMD:C_0603_1608Metric, symbol Device:C
Connections:
- net +3V3: now also C24.1
- net GND: now also C24.2
Changed lines of the file:
@@
 Wire Wire Line
 	4000 3650 4000 3900
+$Comp
+L Device:C C?
+U 1 1 64993225
+P 2250 850
+AR Path="/5F679B53/64993225" Ref="C?"  Part="1"
+AR Path="/5F6B165A/64993225" Ref="C?"  Part="1"
+AR Path="/612D28DD/64993225" Ref="C?"  Part="1"
+AR Path="/61B62C00/64993225" Ref="C?"  Part="1"
+AR Path="/64CBE795/64993225" Ref="C24"  Part="1"
+F 0 "C24" H 2275 950 50  0000 L CNN
+F 1 "100nF" H 2275 750 50  0000 L CNN
+F 2 "Capacitor_SMD:C_0603_1608Metric" H 2288 700 50  0001 C CNN
+F 3 "" H 2250 850 50  0000 C CNN
+F 4 "www.yageo.com" H 2250 850 50  0001 C CNN "MNF1_URL"
+F 5 "CC0603KRX7R9BB104" H 2250 850 50  0001 C CNN "MPN"
+F 6 "603-CC603KRX7R8BB104" H 2250 850 50  0001 C CNN "Mouser"
+F 7 "?" H 2250 850 50  0001 C CNN "Digikey"
+F 8 "" H 2250 850 50  0001 C CNN "LCSC"
+F 9 "?" H 2250 850 50  0001 C CNN "Koncar"
+F 10 "TB" H 2250 850 50  0001 C CNN "Side"
+F 11 "https://www.lcsc.com/product-detail/Multilayer-Ceramic-Capacitors-MLCC-SMD-SMT_YAGEO-CC0603KRX7R9BB104_C14663.html" H 2250 850 50  0001 C CNN "URL"
+	1    2250 850
+	0    1    1    0
+$EndComp
+Wire Wire Line
+	2400 1100 2400 850
+Connection ~ 2400 1100
+Wire Wire Line
+	2100 1100 2100 850
+Connection ~ 2100 1100
 $EndSCHEMATC

Commit message: 3V3 SRAM draft
Parts:
- C20: footprint Capacitor_SMD:C_0603_1608Metric -> Capacitor_SMD:C_0402_1005Metric; MNF1_URL www.yageo.com -> (none); MPN 0603B103K500NT -> CL05B103KB5NNNC; Mouser 603-CC603KRX7R8BB103 -> (none); URL https://www.lcsc.com/product-detail/Multilayer-Ceramic-Capa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 -> (none)
- C22, C23, C24: footprint Capacitor_SMD:C_0603_1608Metric -> Capacitor_SMD:C_0402_1005Metric; MNF1_URL www.yageo.com -> (none); MPN CC0603KRX7R9BB104 -> CL05B104KO5NNNC; Mouser 603-CC603KRX7R8BB104 -> (none); URL https://www.lcsc.com/product-detail/Multilayer-Ceramic-Capa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 -> (none)
Changed lines of the file:
@@
 $Descr A4 11693 8268
 encoding utf-8
-Sheet 4 5
+Sheet 4 6
 Title "nubus-to-ztex HDMI"
 Date ""
@@
 F 0 "C19" H 7325 1800 50  0000 L CNN
 F 1 "100nF" H 7325 1600 50  0000 L CNN
-F 2 "Capacitor_SMD:C_0603_1608Metric" H 7338 1550 50  0001 C CNN
+F 2 "Capacitor_SMD:C_0402_1005Metric" H 7338 1550 50  0001 C CNN
 F 3 "" H 7300 1700 50  0000 C CNN
-F 4 "www.yageo.com" H 7300 1700 50  0001 C CNN "MNF1_URL"
-F 5 "CC0603KRX7R9BB104" H 7300 1700 50  0001 C CNN "MPN"
-F 6 "603-CC603KRX7R8BB104" H 7300 1700 50  0001 C CNN "Mouser"
+F 4 "" H 7300 1700 50  0001 C CNN "MNF1_URL"
+F 5 "CL05B104KO5NNNC" H 7300 1700 50  0001 C CNN "MPN"
+F 6 "" H 7300 1700 50  0001 C CNN "Mouser"
 F 7 "?" H 7300 1700 50  0001 C CNN "Digikey"
 F 8 "" H 7300 1700 50  0001 C CNN "LCSC"
 F 9 "?" H 7300 1700 50  0001 C CNN "Koncar"
 F 10 "TB" H 7300 1700 50  0001 C CNN "Side"
-F 11 "https://www.lcsc.com/product-detail/Multilayer-Ceramic-Capacitors-MLCC-SMD-SMT_YAGEO-CC0603KRX7R9BB104_C14663.html" H 3000 6050 50  0001 C CNN "URL"
+F 11 "" H 3000 6050 50  0001 C CNN "URL"
 	1    7300 1700
 	1    0    0    -1
@@
 F 0 "C17" H 2275 1700 50  0000 L CNN
 F 1 "100nF" H 2275 1500 50  0000 L CNN
-F 2 "Capacitor_SMD:C_0603_1608Metric" H 2288 1450 50  0001 C CNN
+F 2 "Capacitor_SMD:C_0402_1005Metric" H 2288 1450 50  0001 C CNN
 F 3 "" H 2250 1600 50  0000 C CNN
-F 4 "www.yageo.com" H 2250 1600 50  0001 C CNN "MNF1_URL"
-F 5 "CC0603KRX7R9BB104" H 2250 1600 50  0001 C CNN "MPN"
-F 6 "603-CC603KRX7R8BB104" H 2250 1600 50  0001 C CNN "Mouser"
+F 4 "" H 2250 1600 50  0001 C CNN "MNF1_URL"
+F 5 "CL05B104KO5NNNC" H 2250 1600 50  0001 C CNN "MPN"
+F 6 "" H 2250 1600 50  0001 C CNN "Mouser"
 F 7 "?" H 2250 1600 50  0001 C CNN "Digikey"
 F 8 "" H 2250 1600 50  0001 C CNN "LCSC"
 F 9 "?" H 2250 1600 50  0001 C CNN "Koncar"
 F 10 "TB" H 2250 1600 50  0001 C CNN "Side"
-F 11 "https://www.lcsc.com/product-detail/Multilayer-Ceramic-Capacitors-MLCC-SMD-SMT_YAGEO-CC0603KRX7R9BB104_C14663.html" H 2250 1600 50  0001 C CNN "URL"
+F 11 "" H 2250 1600 50  0001 C CNN "URL"
 	1    2250 1600
 	0    1    1    0
@@
 F 0 "C18" H 2475 2000 50  0000 L CNN
 F 1 "100nF" H 2475 1800 50  0000 L CNN
-F 2 "Capacitor_SMD:C_0603_1608Metric" H 2488 1750 50  0001 C CNN
+F 2 "Capacitor_SMD:C_0402_1005Metric" H 2488 1750 50  0001 C CNN
 F 3 "" H 2450 1900 50  0000 C CNN
-F 4 "www.yageo.com" H 2450 1900 50  0001 C CNN "MNF1_URL"
-F 5 "CC0603KRX7R9BB104" H 2450 1900 50  0001 C CNN "MPN"
-F 6 "603-CC603KRX7R8BB104" H 2450 1900 50  0001 C CNN "Mouser"
+F 4 "" H 2450 1900 50  0001 C CNN "MNF1_URL"
+F 5 "CL05B104KO5NNNC" H 2450 1900 50  0001 C CNN "MPN"
+F 6 "" H 2450 1900 50  0001 C CNN "Mouser"
 F 7 "?" H 2450 1900 50  0001 C CNN "Digikey"
 F 8 "" H 2450 1900 50  0001 C CNN "LCSC"
 F 9 "?" H 2450 1900 50  0001 C CNN "Koncar"
 F 10 "TB" H 2450 1900 50  0001 C CNN "Side"
-F 11 "https://www.lcsc.com/product-detail/Multilayer-Ceramic-Capacitors-MLCC-SMD-SMT_YAGEO-CC0603KRX7R9BB104_C14663.html" H 3000 6050 50  0001 C CNN "URL"
+F 11 "" H 3000 6050 50  0001 C CNN "URL"
 	1    2450 1900
 	0    1    1    0
@@
 F 0 "C15" H 2275 1200 50  0000 L CNN
 F 1 "10nF" H 2275 1000 50  0000 L CNN
-F 2 "Capacitor_SMD:C_0603_1608Metric" H 2288 950 50  0001 C CNN
+F 2 "Capacitor_SMD:C_0402_1005Metric" H 2288 950 50  0001 C CNN
 F 3 "" H 2250 1100 50  0000 C CNN
-F 4 "www.yageo.com" H 2250 1100 50  0001 C CNN "MNF1_URL"
-F 5 "0603B103K500NT" H 2250 1100 50  0001 C CNN "MPN"
-F 6 "603-CC603KRX7R8BB103" H 2250 1100 50  0001 C CNN "Mouser"
-F 7 "https://www.lcsc.com/product-detail/Multilayer-Ceramic-Capacitors-MLCC-SMD-SMT_FH-Guangdong-Fenghua-Advanced-Tech-0603B103K500NT_C57112.html" H 2250 1100 50  0001 C CNN "URL"
+F 4 "" H 2250 1100 50  0001 C CNN "MNF1_URL"
+F 5 "CL05B103KB5NNNC" H 2250 1100 50  0001 C CNN "MPN"
+F 6 "" H 2250 1100 50  0001 C CNN "Mouser"
+F 7 "" H 2250 1100 50  0001 C CNN "URL"
 	1    2250 1100
 	0    1    1    0
@@
 F 0 "C24" H 2275 950 50  0000 L CNN
 F 1 "100nF" H 2275 750 50  0000 L CNN
-F 2 "Capacitor_SMD:C_0603_1608Metric" H 2288 700 50  0001 C CNN
+F 2 "Capacitor_SMD:C_0402_1005Metric" H 2288 700 50  0001 C CNN
 F 3 "" H 2250 850 50  0000 C CNN
-F 4 "www.yageo.com" H 2250 850 50  0001 C CNN "MNF1_URL"
-F 5 "CC0603KRX7R9BB104" H 2250 850 50  0001 C CNN "MPN"
-F 6 "603-CC603KRX7R8BB104" H 2250 850 50  0001 C CNN "Mouser"
+F 4 "" H 2250 850 50  0001 C CNN "MNF1_URL"
+F 5 "CL05B104KO5NNNC" H 2250 850 50  0001 C CNN "MPN"
+F 6 "" H 2250 850 50  0001 C CNN "Mouser"
 F 7 "?" H 2250 850 50  0001 C CNN "Digikey"
 F 8 "" H 2250 850 50  0001 C CNN "LCSC"
 F 9 "?" H 2250 850 50  0001 C CNN "Koncar"
 F 10 "TB" H 2250 850 50  0001 C CNN "Side"
-F 11 "https://www.lcsc.com/product-detail/Multilayer-Ceramic-Capacitors-MLCC-SMD-SMT_YAGEO-CC0603KRX7R9BB104_C14663.html" H 2250 850 50  0001 C CNN "URL"
+F 11 "" H 2250 850 50  0001 C CNN "URL"
 	1    2250 850
 	0    1    1    0
