File: IIsi-to-ztex/pmod.sch (KiCad schematic (older format))
At the start: 10 parts, among them J4 A2541HWR-2x6P (Pmod 2x6 F R)

Commit message: 3V3 SRAM draft
Parts:
- C15: footprint Capacitor_SMD:C_0603_1608Metric -> Capacitor_SMD:C_0402_1005Metric; MNF1_URL www.yageo.com -> (none); MPN CC0603KRX7R9BB104 -> CL05B104KO5NNNC; Mouser 603-CC603KRX7R8BB104 -> (none); URL https://www.lcsc.com/product-detail/Multilayer-Ceramic-Capa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 -> (none)
Changed lines of the file:
@@
 $Descr A4 11693 8268
 encoding utf-8
-Sheet 5 5
+Sheet 5 6
 Title "sbus-to-ztex blinkey stuff"
 Date ""
@@
 F 0 "C21" H 8175 3350 50  0000 L CNN
 F 1 "100nF" H 8175 3150 50  0000 L CNN
-F 2 "Capacitor_SMD:C_0603_1608Metric" H 8188 3100 50  0001 C CNN
+F 2 "Capacitor_SMD:C_0402_1005Metric" H 8188 3100 50  0001 C CNN
 F 3 "" H 8150 3250 50  0000 C CNN
-F 4 "www.yageo.com" H 8150 3250 50  0001 C CNN "MNF1_URL"
-F 5 "CC0603KRX7R9BB104" H 8150 3250 50  0001 C CNN "MPN"
-F 6 "603-CC603KRX7R8BB104" H 8150 3250 50  0001 C CNN "Mouser"
+F 4 "" H 8150 3250 50  0001 C CNN "MNF1_URL"
+F 5 "CL05B104KO5NNNC" H 8150 3250 50  0001 C CNN "MPN"
+F 6 "" H 8150 3250 50  0001 C CNN "Mouser"
 F 7 "?" H 8150 3250 50  0001 C CNN "Digikey"
 F 8 "" H 8150 3250 50  0001 C CNN "LCSC"
 F 9 "?" H 8150 3250 50  0001 C CNN "Koncar"
 F 10 "TB" H 8150 3250 50  0001 C CNN "Side"
-F 11 "https://www.lcsc.com/product-detail/Multilayer-Ceramic-Capacitors-MLCC-SMD-SMT_YAGEO-CC0603KRX7R9BB104_C14663.html" H 3000 6050 50  0001 C CNN "URL"
+F 11 "" H 3000 6050 50  0001 C CNN "URL"
 	1    8150 3250
 	1    0    0    -1
