File: IIsiA7_Mini/board_specific.kicad_sch (KiCad schematic)
At the start: 6 parts, among them J5 USB Micro-B, U7 74LVC1G125DRL

Commit message: fix BoM
Parts:
- U7: value 74LVC1G125DRL -> 74LVC1G125DCK; MPN SN74LVC1G125DRLR-TP -> SN74LVC1G125DCKR
Changed lines of the file:
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@@
 			)
 		)
-		(property "Value" "74LVC1G125DRL"
+		(property "Value" "74LVC1G125DCK"
 			(at 209.2741 102.8577 0)
 			(effects
@@
 			)
 		)
-		(property "MPN" "SN74LVC1G125DRLR-TP"
+		(property "MPN" "SN74LVC1G125DCKR"
 			(at 195.58 106.68 0)
 			(effects
